File: terrarium shield.brd (EAGLE design)
At the start: 68.6 x 53.3 mm, 17 parts

Commit message: Connected the other two GND pins to the ground pour.
Connections:
- removed net GND1: U$1.GND1
- net GND: now also U$1.GND1
Changed lines of the file:
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@@
 </polygon>
 <contactref element="C2" pad="2"/>
-<contactref element="U$1" pad="GND"/>
 <contactref element="PILLAR4" pad="GND"/>
 <contactref element="PILLAR3" pad="GND"/>
@@
 <contactref element="TEMP_HUM" pad="GND"/>
 <contactref element="RESET" pad="T1"/>
+<contactref element="U$1" pad="GND1"/>
+<contactref element="U$1" pad="GND"/>
 </signal>
 <signal name="+5V" class="1">
@@
 <wire x1="33.02" y1="5.08" x2="33.02" y2="2.54" width="0.762" layer="1"/>
 </signal>
-<signal name="GND1">
-<contactref element="U$1" pad="GND1"/>
-</signal>
 <signal name="5V">

Commit message: Removed DC jack. Will get power from VIN.
Parts:
- removed 5V_DC: 2.1MM_DC_JACK, tjw:2.1MM_DC_JACK
Connections:
- net +5V: no longer 5V_DC.+V
- net GND: no longer 5V_DC.GND
Routing:
- net +5V: track 164.8 -> 161.4 mm
Changed lines of the file:
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@@
 <layers>
 <layer number="1" name="Top" color="4" fill="1" visible="yes" active="yes"/>
-<layer number="16" name="Bottom" color="1" fill="1" visible="yes" active="yes"/>
+<layer number="16" name="Bottom" color="1" fill="1" visible="no" active="yes"/>
 <layer number="17" name="Pads" color="2" fill="1" visible="yes" active="yes"/>
 <layer number="18" name="Vias" color="2" fill="1" visible="yes" active="yes"/>
@@
 <element name="C2" library="SparkFun-Passives" package="CPOL-RADIAL-1000UF-25V" value="1000uF" x="39.37" y="10.16"/>
 <element name="U$1" library="tjw" package="ARDUINO_UNO_R3" value="ARDUINO_UNO_R3" x="0" y="0"/>
-<element name="5V_DC" library="tjw" package="2.1MM_DC_JACK" value="2.1MM_DC_JACK" x="15.24" y="21.59" smashed="yes" rot="R90">
-<attribute name="NAME" x="8.89" y="20.32" size="1.27" layer="21" rot="R180"/>
-</element>
 <element name="TEMP_HUM" library="tjw" package="MOLEX_3PIN_VERT_THM" value="MOLEX_3PIN_VERT_THM" x="22.86" y="34.29" rot="R90"/>
 <element name="LED0" library="tjw" package="MOLEX_3PIN_VERT_THM" value="MOLEX_3PIN_VERT_THM" x="22.86" y="22.86" rot="R90"/>
@@
 <signal name="GND" class="1">
 <contactref element="U$1" pad="GND2"/>
-<contactref element="5V_DC" pad="GND"/>
 <polygon width="0.254" layer="16">
 <vertex x="1.27" y="52.07"/>
@@
 <signal name="+5V" class="1">
 <contactref element="U$1" pad="VIN"/>
-<contactref element="5V_DC" pad="+V"/>
 <contactref element="C2" pad="1"/>
 <contactref element="PILLAR4" pad="+V"/>
@@
 <wire x1="18.91" y1="18.74" x2="18.91" y2="24.81" width="0.762" layer="1"/>
 <wire x1="18.91" y1="24.81" x2="19.36" y2="25.26" width="0.762" layer="1"/>
-<wire x1="19.36" y1="25.26" x2="15.47" y2="25.26" width="0.762" layer="1"/>
-<wire x1="15.47" y1="25.26" x2="14.54" y2="26.19" width="0.762" layer="1"/>
 <wire x1="19.36" y1="36.69" x2="18.91" y2="36.69" width="0.762" layer="1"/>
-<wire x1="18.91" y1="36.69" x2="16.51" y2="34.29" width="0.762" layer="1"/>
-<wire x1="16.51" y1="34.29" x2="16.51" y2="28.16" width="0.762" layer="1"/>
-<wire x1="16.51" y1="28.16" x2="14.54" y2="26.19" width="0.762" layer="1"/>
 <contactref element="R2" pad="P$2"/>
 <wire x1="31.61" y1="21.28" x2="31.61" y2="15.38" width="0.762" layer="1"/>
@@
 <wire x1="14.07" y1="15.87" x2="18.41" y2="15.87" width="0.762" layer="1"/>
 <wire x1="18.41" y1="15.87" x2="19.05" y2="16.51" width="0.762" layer="1"/>
+<wire x1="18.91" y1="36.69" x2="16.51" y2="34.29" width="0.762" layer="1"/>
+<wire x1="16.51" y1="34.29" x2="16.51" y2="26.84" width="0.762" layer="1"/>
+<wire x1="16.51" y1="26.84" x2="19.36" y2="25.26" width="0.762" layer="1"/>
 </signal>
 <signal name="N$13">
