File: terrarium board.brd (EAGLE design)
At the start: 84.8 x 80 mm, 30 parts

Commit message: Sadly, pillar0 was touching, but Eagle didn't think it was hooked up.
Connections:
- net N$26: now also SPARK.D6
Changed lines of the file:
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@@
 <signal name="N$26">
 <contactref element="SHIFT2" pad="13"/>
+<contactref element="SPARK" pad="D6"/>
+<wire x1="16.1815" y1="40.745" x2="25.285" y2="47.84" width="0" layer="19" extent="1-1"/>
 </signal>
 </signals>

Commit message: Fixed issues from v2.
Parts:
- moved C3 9.96 mm to (33.5, 46.7), turned to 270 degrees
- moved SHIFT2 6.30 mm to (22.2, 52.8)
- moved R1 1.40 mm to (76.6, 17.3)
- moved R6 1.20 mm to (75.4, 64.7)
- moved R4 0.80 mm to (36.5, 15.7)
- moved R2 0.70 mm to (62.6, 17.0)
- moved R3 0.70 mm to (50.5, 15.9)
Routing:
- net +5V: track 357.5 -> 338.5 mm
- net GND: track 96.7 -> 110.2 mm
- net N$26: track 0.00 -> 7.68 mm
- net N$13: track 33.2 -> 38.9 mm
- net N$15: track 21.3 -> 26.9 mm
- net N$25: track 19.8 -> 14.5 mm
- net N$10: track 46.1 -> 50.8 mm
- net N$23: track 10.4 -> 14.7 mm
- net N$32: track 11.5 -> 7.35 mm
- net N$33: track 10.3 -> 7.21 mm
- net N$31: track 9.29 -> 7.19 mm
- net N$4: track 4.89 -> 6.78 mm
- net N$24: track 8.19 -> 6.46 mm
- net N$22: track 28.3 -> 26.8 mm
- net N$5: track 26.3 -> 24.8 mm
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Other:
- board text added: "Terrarium v2.1"
- board text removed: "Terrarium v2"
